File: kicad-stomp/stomp-board.kicad_pcb (KiCad board)
At the start: 2 copper layers, 19 x 20.5 mm, 2 parts, among them J1 Conn_01x06, SW1 SW_3PDT_x3

Commit message: Prodfiles for stomp
Routing:
- net /STOMP_OUT_GND: track 13.5 -> 12.3 mm
- net /STOMP_OUT_R: track 18.0 -> 17.3 mm
- net /STOMP_OUT_L: track 22.9 -> 22.3 mm
- net /DRY_IN_R: track 22.5 -> 22.0 mm
- added copper zone on B.Cu, net (none)
- added copper zone on F.Cu, net (none)
Changed lines of the file:
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@@
 		(tenting front back)
 		(pcbplotparams
-			(layerselection 0x00000000_00000000_55555555_5755f5ff)
+			(layerselection 0x00000000_00000000_55555555_57555555)
 			(plot_on_all_layers_selection 0x00000000_00000000_00000000_00000000)
 			(disableapertmacros no)
@@
 			(psa4output no)
 			(plot_black_and_white yes)
+			(plotinvisibletext no)
 			(sketchpadsonfab no)
 			(plotpadnumbers no)
@@
 			(outputformat 1)
 			(mirror no)
-			(drillshape 1)
+			(drillshape 0)
 			(scaleselection 1)
-			(outputdirectory "")
+			(outputdirectory "prod_files/")
 		)
 	)
@@
 	)
 	(segment
-		(start 116.15 101.4)
-		(end 116.15 111.15)
-		(width 0.2)
+		(start 116.248 111.248)
+		(end 118.5 113.5)
+		(width 0.3)
 		(layer "F.Cu")
 		(net 1)
@@
 	(segment
 		(start 124.35 98.4)
-		(end 122.96645 99.78355)
-		(width 0.2)
+		(end 121.852 100.898)
+		(width 0.3)
 		(layer "F.Cu")
 		(net 1)
 	)
 	(segment
-		(start 116.15 111.15)
-		(end 118.5 113.5)
-		(width 0.2)
+		(start 116.248 102.070745)
+		(end 116.248 111.248)
+		(width 0.3)
 		(layer "F.Cu")
 		(net 1)
 	)
 	(segment
-		(start 122.96645 99.78355)
-		(end 117.76645 99.78355)
-		(width 0.2)
+		(start 121.852 100.898)
+		(end 117.420745 100.898)
+		(width 0.3)
 		(layer "F.Cu")
 		(net 1)
 	)
 	(segment
-		(start 117.76645 99.78355)
-		(end 116.15 101.4)
-		(width 0.2)
+		(start 117.420745 100.898)
+		(end 116.248 102.070745)
+		(width 0.3)
 		(layer "F.Cu")
 		(net 1)
+	)
+	(segment
+		(start 124.35 107.5)
+		(end 124.35 113.35)
+		(width 0.3)
+		(layer "F.Cu")
+		(net 2)
 	)
 	(segment
 		(start 124.35 113.35)
 		(end 124.5 113.5)
-		(width 0.2)
+		(width 0.3)
 		(layer "F.Cu")
 		(net 2)
 	)
 	(segment
-		(start 124.35 107.5)
-		(end 124.35 113.35)
-		(width 0.2)
-		(layer "F.Cu")
-		(net 2)
-	)
-	(segment
-		(start 118.2 98.3)
-		(end 115.5 101)
-		(width 0.2)
+		(start 117.300001 98.3)
+		(end 115.647 99.953001)
+		(width 0.3)
 		(layer "F.Cu")
 		(net 3)
 	)
 	(segment
-		(start 115.5 112.5)
+		(start 115.647 112.647)
 		(end 116.5 113.5)
-		(width 0.2)
+		(width 0.3)
 		(layer "F.Cu")
 		(net 3)
 	)
 	(segment
-		(start 115.5 101)
-		(end 115.5 112.5)
-		(width 0.2)
+		(start 119.2 98.3)
+		(end 117.300001 98.3)
+		(width 0.3)
 		(layer "F.Cu")
 		(net 3)
 	)
 	(segment
-		(start 119.2 98.3)
-		(end 118.2 98.3)
-		(width 0.2)
+		(start 115.647 99.953001)
+		(end 115.647 112.647)
+		(width 0.3)
 		(layer "F.Cu")
 		(net 3)
 	)
 	(segment
-		(start 131.95 110.05)
+		(start 131.851 110.149)
 		(end 128.5 113.5)
-		(width 0.2)
+		(width 0.3)
 		(layer "F.Cu")
 		(net 4)
 	)
 	(segment
-		(start 120.85 102.9)
-		(end 123 105.05)
-		(width 0.2)
+		(start 122.399 106.099)
+		(end 131.030313 106.099)
+		(width 0.3)
 		(layer "F.Cu")
 		(net 4)
 	)
 	(segment
-		(start 130.9 105.05)
-		(end 131.95 106.1)
-		(width 0.2)
+		(start 119.2 102.9)
+		(end 122.399 106.099)
+		(width 0.3)
 		(layer "F.Cu")
 		(net 4)
 	)
 	(segment
-		(start 131.95 106.1)
-		(end 131.95 110.05)
-		(width 0.2)
+		(start 131.851 106.919687)
+		(end 131.851 110.149)
+		(width 0.3)
 		(layer "F.Cu")
 		(net 4)
 	)
 	(segment
-		(start 123 105.05)
-		(end 130.9 105.05)
-		(width 0.2)
+		(start 131.030313 106.099)
+		(end 131.851 106.919687)
+		(width 0.3)
 		(layer "F.Cu")
 		(net 4)
 	)
 	(segment
-		(start 119.2 102.9)
-		(end 120.85 102.9)
-		(width 0.2)
-		(layer "F.Cu")
-		(net 4)
-	)
-	(segment
-		(start 131.65 102.9)
-		(end 133 104.25)
-		(width 0.2)
+		(start 129.5 102.9)
+		(end 129.531197 102.9)
+		(width 0.3)
 		(layer "F.Cu")
 		(net 5)
 	)
 	(segment
-		(start 129.5 102.9)
-		(end 131.65 102.9)
-		(width 0.2)
+		(start 133.053 106.421803)
+		(end 133.053 112.947)
+		(width 0.3)
 		(layer "F.Cu")
 		(net 5)
 	)
 	(segment
-		(start 133 113)
+		(start 129.531197 102.9)
+		(end 133.053 106.421803)
+		(width 0.3)
+		(layer "F.Cu")
+		(net 5)
+	)
+	(segment
+		(start 133.053 112.947)
 		(end 132.5 113.5)
-		(width 0.2)
+		(width 0.3)
 		(layer "F.Cu")
 		(net 5)
 	)
 	(segment
-		(start 133 104.25)
-		(end 133 113)
-		(width 0.2)
-		(layer "F.Cu")
-		(net 5)
-	)
-	(segment
-		(start 126 102.9)
-		(end 127.5 104.4)
-		(width 0.2)
+		(start 126.948 105.498)
+		(end 131.279255 105.498)
+		(width 0.3)
 		(layer "F.Cu")
 		(net 6)
 	)
 	(segment
-		(start 132.5 105.55)
-		(end 132.5 111.5)
-		(width 0.2)
+		(start 131.279255 105.498)
+		(end 132.452 106.670745)
+		(width 0.3)
 		(layer "F.Cu")
 		(net 6)
 	)
 	(segment
+		(start 132.452 111.548)
+		(end 130.5 113.5)
+		(width 0.3)
+		(layer "F.Cu")
+		(net 6)
+	)
+	(segment
+		(start 132.452 106.670745)
+		(end 132.452 111.548)
+		(width 0.3)
+		(layer "F.Cu")
+		(net 6)
+	)
+	(segment
 		(start 124.35 102.9)
-		(end 126 102.9)
-		(width 0.2)
+		(end 126.948 105.498)
+		(width 0.3)
 		(layer "F.Cu")
 		(net 6)
 	)
 	(segment
-		(start 131.35 104.4)
-		(end 132.5 105.55)
-		(width 0.2)
-		(layer "F.Cu")
-		(net 6)
-	)
-	(segment
-		(start 127.5 104.4)
-		(end 131.35 104.4)
-		(width 0.2)
-		(layer "F.Cu")
-		(net 6)
-	)
-	(segment
-		(start 132.5 111.5)
-		(end 130.5 113.5)
-		(width 0.2)
-		(layer "F.Cu")
-		(net 6)
+		(start 129.5 107.5)
+		(end 129.5 110.5)
+		(width 0.3)
+		(layer "F.Cu")
+		(net 7)
 	)
 	(segment
 		(start 129.5 110.5)
 		(end 126.5 113.5)
-		(width 0.2)
+		(width 0.3)
 		(layer "F.Cu")
 		(net 7)
 	)
 	(segment
-		(start 129.5 107.5)
-		(end 129.5 110.5)
-		(width 0.2)
-		(layer "F.Cu")
-		(net 7)
-	)
-	(segment
 		(start 129.5 98.4)
-		(end 127.5 100.4)
-		(width 0.2)
+		(end 126.401 101.499)
+		(width 0.3)
 		(layer "F.Cu")
 		(net 8)
 	)
 	(segment
-		(start 127.5 100.4)
-		(end 118.35 100.4)
-		(width 0.2)
+		(start 126.401 101.499)
+		(end 117.669687 101.499)
+		(width 0.3)
 		(layer "F.Cu")
 		(net 8)
 	)
 	(segment
-		(start 118.35 100.4)
-		(end 116.85 101.9)
-		(width 0.2)
+		(start 117.669687 101.499)
+		(end 116.849 102.319687)
+		(width 0.3)
 		(layer "F.Cu")
 		(net 8)
 	)
 	(segment
-		(start 116.85 101.9)
-		(end 116.85 109.85)
-		(width 0.2)
+		(start 116.849 109.849)
+		(end 120.5 113.5)
+		(width 0.3)
 		(layer "F.Cu")
 		(net 8)
 	)
 	(segment
-		(start 116.85 109.85)
-		(end 120.5 113.5)
-		(width 0.2)
+		(start 116.849 102.319687)
+		(end 116.849 109.849)
+		(width 0.3)
 		(layer "F.Cu")
 		(net 8)
+	)
+	(segment
+		(start 119.2 110.2)
+		(end 122.5 113.5)
+		(width 0.3)
+		(layer "F.Cu")
+		(net 9)
 	)
 	(segment
 		(start 119.2 107.5)
 		(end 119.2 110.2)
-		(width 0.2)
+		(width 0.3)
 		(layer "F.Cu")
 		(net 9)
 	)
-	(segment
-		(start 119.2 110.2)
-		(end 122.5 113.5)
-		(width 0.2)
-		(layer "F.Cu")
-		(net 9)
+	(zone
+		(net 0)
+		(net_name "")
+		(layers "F.Cu" "B.Cu")
+		(hatch edge 0.5)
+		(connect_pads
+			(clearance 0.5)
+		)
+		(min_thickness 0.25)
+		(filled_areas_thickness no)
+		(fill yes
+			(thermal_gap 0.5)
+			(thermal_bridge_width 0.5)
+			(island_removal_mode 1)
+			(island_area_min 10)
+		)
+		(polygon
+			(pts
+				(xy 134.5 115.5) (xy 114.5 115.5) (xy 114.5 93.75) (xy 134.5 93.75) (xy 134.5 93.75)
+			)
+		)
 	)
 	(embedded_fonts no)
